Commit message: fixed urdf motor initial degree

File: single_arm_6dof_description/urdf/single_arm_6dof.xacro (robot description, xacro)
@@ -13,15 +13,15 @@
     <inertial>
       <origin
-        xyz="-0.00015623 -0.00020293 0.064403"
-        rpy="0 0 0" />
-      <mass
-        value="0.47718" />
-      <inertia
-        ixx="0.00059054"
+        xyz="-3.4663E-05 -4.5026E-05 0.0084004"
+        rpy="0 0 0" />
+      <mass
+        value="2.1507" />
+      <inertia
+        ixx="0.0094824"
         ixy="3.555E-10"
         ixz="-4.1821E-06"
-        iyy="0.00059015"
+        iyy="0.0095713"
         iyz="-9.8398E-08"
-        izz="0.00022102" />
+        izz="0.018031" />
     </inertial>
     <visual>
@@ -67,15 +67,15 @@
     <inertial>
       <origin
-        xyz="3.30503515696967E-06 0.00361463453669447 0.0290846870786987"
-        rpy="0 0 0" />
-      <mass
-        value="0.402880268420354" />
-      <inertia
-        ixx="0.000481117385082944"
-        ixy="-7.08270540835146E-08"
-        ixz="-3.55657214762967E-10"
-        iyy="0.000189861333802929"
-        iyz="4.18208632570024E-06"
-        izz="0.000494803815076241" />
+        xyz="3.305E-06 0.0036146 0.029085"
+        rpy="0 0 0" />
+      <mass
+        value="0.40288" />
+      <inertia
+        ixx="0.00048112"
+        ixy="-7.0827E-08"
+        ixz="-3.5566E-10"
+        iyy="0.00018986"
+        iyz="4.1821E-06"
+        izz="0.0004948" />
     </inertial>
     <visual>
@@ -121,15 +121,15 @@
     <inertial>
       <origin
-        xyz="-2.63459088767348E-07 0.172940222302508 0.00052652750922403"
-        rpy="0 0 0" />
-      <mass
-        value="0.602986093363339" />
-      <inertia
-        ixx="0.000747867407695296"
-        ixy="1.95782582360181E-12"
-        ixz="4.26723886970973E-10"
-        iyy="0.000502016615573157"
-        iyz="3.67313449365761E-07"
-        izz="0.000474271843381996" />
+        xyz="-2.4369E-07 0.18004 0.0061614"
+        rpy="0 0 0" />
+      <mass
+        value="0.6519" />
+      <inertia
+        ixx="0.00076385"
+        ixy="2.1135E-12"
+        ixz="4.2672E-10"
+        iyy="0.00051784"
+        iyz="3.6733E-07"
+        izz="0.00050582" />
     </inertial>
     <visual>
@@ -162,5 +162,5 @@
     <origin
       xyz="0 0.2675 -0.039"
-      rpy="-3.1416 0 1.5708" />
+      rpy="-3.1416 0 3.1416" />
     <parent
       link="link2" />
@@ -178,15 +178,15 @@
     <inertial>
       <origin
-        xyz="2.22805200233989E-07 0.153208866547273 0.00308035588048404"
-        rpy="0 0 0" />
-      <mass
-        value="0.571051286792162" />
-      <inertia
-        ixx="0.000589782400801251"
-        ixy="-1.02113667044765E-11"
-        ixz="9.04380132437654E-10"
-        iyy="0.000451003170410362"
-        iyz="1.25771372588246E-06"
-        izz="0.000358850501032578" />
+        xyz="2.2281E-07 0.15321 0.0030804"
+        rpy="0 0 0" />
+      <mass
+        value="0.57105" />
+      <inertia
+        ixx="0.00058978"
+        ixy="-1.0211E-11"
+        ixz="9.0438E-10"
+        iyy="0.000451"
+        iyz="1.2577E-06"
+        izz="0.00035885" />
     </inertial>
     <visual>
@@ -234,15 +234,15 @@
     <inertial>
       <origin
-        xyz="0.010389914754231 -1.66533453693773E-16 0.0240404001873197"
-        rpy="0 0 0" />
-      <mass
-        value="0.159189766593809" />
-      <inertia
-        ixx="4.47597165263928E-05"
-        ixy="-1.07719622601504E-19"
-        ixz="5.33461873898255E-07"
-        iyy="9.4187030469331E-05"
-        iyz="1.45020014212472E-16"
-        izz="0.000102703497027636" />
+        xyz="0.01039 -1.3878E-16 0.02404"
+        rpy="0 0 0" />
+      <mass
+        value="0.15919" />
+      <inertia
+        ixx="4.476E-05"
+        ixy="-1.095E-19"
+        ixz="5.3346E-07"
+        iyy="9.4187E-05"
+        iyz="1.4501E-16"
+        izz="0.0001027" />
     </inertial>
     <visual>
@@ -274,5 +274,5 @@
     <origin
       xyz="0.052 0 0.0286"
-      rpy="1.5708 0 1.5708" />
+      rpy="0 1.5708 0" />
     <parent
       link="link4" />
@@ -290,15 +290,15 @@
     <inertial>
       <origin
-        xyz="-0.0104572514863331 1.38777878078145E-16 0.0286143000684295"
-        rpy="0 0 0" />
-      <mass
-        value="0.158164705784998" />
-      <inertia
-        ixx="4.3878104420964E-05"
-        ixy="-1.00184733759959E-19"
-        ixz="-5.33461873898271E-07"
-        iyy="9.36578426684008E-05"
-        iyz="-1.45012495530806E-16"
-        izz="0.000101330258427024" />
+        xyz="-0.010457 8.3267E-17 0.028614"
+        rpy="0 0 0" />
+      <mass
+        value="0.15816" />
+      <inertia
+        ixx="4.3878E-05"
+        ixy="-1.249E-19"
+        ixz="-5.3346E-07"
+        iyy="9.3658E-05"
+        iyz="-1.4501E-16"
+        izz="0.00010133" />
     </inertial>
     <visual>
@@ -331,5 +331,5 @@
     <origin
       xyz="-0.055 0 0.033001"
-      rpy="3.1416 -1.5708 0" />
+      rpy="0 -1.5708 0" />
     <parent
       link="link5" />
@@ -347,15 +347,15 @@
     <inertial>
       <origin
-        xyz="-5.37938103728486E-07 -2.77555756156289E-17 0.00700006055550928"
-        rpy="0 0 0" />
-      <mass
-        value="0.0259770442543706" />
-      <inertia
-        ixx="2.20534281951168E-06"
-        ixy="1.54848210669926E-22"
-        ixz="2.93316535498093E-21"
-        iyy="2.20534281951168E-06"
-        iyz="-4.44622696747536E-22"
-        izz="3.97773490145051E-06" />
+        xyz="-5.3794E-07 4.1633E-16 0.0070001"
+        rpy="0 0 0" />
+      <mass
+        value="0.025977" />
+      <inertia
+        ixx="2.2053E-06"
+        ixy="2.5014E-22"
+        ixz="-1.4272E-22"
+        iyy="2.2053E-06"
+        iyz="-1.2285E-22"
+        izz="3.9777E-06" />
     </inertial>
     <visual>
